File: CurrentSense.sch (KiCad schematic (older format))
At the start: 7 parts, among them U5 INA139, U7 OPA340NA

Commit message: Lots of routing done
Connections:
- net labels added: +3V3_2
- net labels removed: +3V3
Changed lines of the file:
@@
 	6550 3200 6550 3700
-$Comp
-L power:+3V3 #PWR0113
-U 1 1 60490764
-P 6150 3400
-F 0 "#PWR0113" H 6150 3250 50  0001 C CNN
-F 1 "+3V3" H 6250 3500 50  0000 C CNN
-F 2 "" H 6150 3400 50  0001 C CNN
-F 3 "" H 6150 3400 50  0001 C CNN
-	1    6150 3400
-	1    0    0    -1
-$EndComp
 $Comp
 L power:GND #PWR0132
@@
 	0    1    1    0
 $EndComp
+$Comp
+L power:+3V3_2 #PWR?
+U 1 1 61134136
+P 6150 3400
+F 0 "#PWR?" H 6150 3250 50  0001 C CNN
+F 1 "+3V3_2" H 6300 3500 50  0000 C CNN
+F 2 "" H 6150 3400 50  0001 C CNN
+F 3 "" H 6150 3400 50  0001 C CNN
+	1    6150 3400
+	1    0    0    -1
+$EndComp
 $EndSCHEMATC
