File: MCU_2.sch (KiCad schematic (older format))
At the start: 18 parts, among them U6 STM32F051K6Ux

Commit message: Lots of routing done
Connections:
- net labels added: +3V3_2
- net labels removed: +3V3
Changed lines of the file:
@@
 $EndComp
 $Comp
-L power:+3V3 #PWR?
-U 1 1 6059DC2C
-P 3800 1700
-AR Path="/6059DC2C" Ref="#PWR?"  Part="1"
-AR Path="/60302A40/6059DC2C" Ref="#PWR0101"  Part="1"
-AR Path="/605793E5/6059DC2C" Ref="#PWR0149"  Part="1"
-AR Path="/6057AB62/6059DC2C" Ref="#PWR?"  Part="1"
-AR Path="/6054D32F/6059DC2C" Ref="#PWR0111"  Part="1"
-AR Path="/60568CD3/6059DC2C" Ref="#PWR?"  Part="1"
-AR Path="/60575054/6059DC2C" Ref="#PWR?"  Part="1"
-AR Path="/60595215/6059DC2C" Ref="#PWR0182"  Part="1"
-AR Path="/605A2EB9/6059DC2C" Ref="#PWR0207"  Part="1"
-AR Path="/60535FFC/6059DC2C" Ref="#PWR0180"  Part="1"
-AR Path="/6072B375/6059DC2C" Ref="#PWR0138"  Part="1"
-AR Path="/6077FA6E/6059DC2C" Ref="#PWR0153"  Part="1"
-AR Path="/60799273/6059DC2C" Ref="#PWR0153"  Part="1"
-F 0 "#PWR0138" H 3800 1550 50  0001 C CNN
-F 1 "+3V3" H 3815 1873 50  0000 C CNN
-F 2 "" H 3800 1700 50  0001 C CNN
-F 3 "" H 3800 1700 50  0001 C CNN
-	1    3800 1700
-	1    0    0    -1
-$EndComp
-$Comp
 L power:GND #PWR?
 U 1 1 6059DC2D
@@
 	1    0    0    -1
 $EndComp
-Connection ~ 3800 1700
 Connection ~ 3800 1900
 Wire Wire Line
@@
 NRST
 $Comp
-L power:+3V3 #PWR0110
-U 1 1 6059DC35
-P 5400 1450
-AR Path="/60302A40/6059DC35" Ref="#PWR0110"  Part="1"
-AR Path="/605793E5/6059DC35" Ref="#PWR0157"  Part="1"
-AR Path="/6057AB62/6059DC35" Ref="#PWR?"  Part="1"
-AR Path="/6054D32F/6059DC35" Ref="#PWR0161"  Part="1"
-AR Path="/60568CD3/6059DC35" Ref="#PWR?"  Part="1"
-AR Path="/60575054/6059DC35" Ref="#PWR?"  Part="1"
-AR Path="/60595215/6059DC35" Ref="#PWR0190"  Part="1"
-AR Path="/605A2EB9/6059DC35" Ref="#PWR0219"  Part="1"
-AR Path="/60535FFC/6059DC35" Ref="#PWR0188"  Part="1"
-AR Path="/6072B375/6059DC35" Ref="#PWR0145"  Part="1"
-AR Path="/6077FA6E/6059DC35" Ref="#PWR0161"  Part="1"
-AR Path="/60799273/6059DC35" Ref="#PWR0161"  Part="1"
-F 0 "#PWR0145" H 5400 1300 50  0001 C CNN
-F 1 "+3V3" H 5300 1600 50  0000 C CNN
-F 2 "" H 5400 1450 50  0001 C CNN
-F 3 "" H 5400 1450 50  0001 C CNN
-	1    5400 1450
-	1    0    0    -1
-$EndComp
-$Comp
 L Device:C_Small C?
 U 1 1 604562F9
@@
 AR Path="/60799273/6056D000" Ref="#PWR0166"  Part="1"
 F 0 "#PWR0149" H 6100 1400 50  0001 C CNN
-F 1 "+3V3A_2" H 6085 1623 50  0000 C CNN
+F 1 "+3V3A_2" H 6250 1600 50  0000 C CNN
 F 2 "" H 6100 1450 50  0001 C CNN
 F 3 "" H 6100 1450 50  0001 C CNN
@@
 AR Path="/60799273/6078D9AE" Ref="#PWR?"  Part="1"
 F 0 "#PWR0136" H 5250 1950 50  0001 C CNN
-F 1 "+3V3A_2" H 5235 2173 50  0000 C CNN
+F 1 "+3V3A_2" H 5350 2150 50  0000 C CNN
 F 2 "" H 5250 2000 50  0001 C CNN
 F 3 "" H 5250 2000 50  0001 C CNN
@@
 $EndComp
 $Comp
-L power:+3V3 #PWR?
-U 1 1 607587D5
-P 5050 2000
-AR Path="/60302A40/607587D5" Ref="#PWR?"  Part="1"
-AR Path="/605793E5/607587D5" Ref="#PWR?"  Part="1"
-AR Path="/6054D32F/607587D5" Ref="#PWR?"  Part="1"
-AR Path="/605CA831/607587D5" Ref="#PWR?"  Part="1"
-AR Path="/6073F35C/607587D5" Ref="#PWR?"  Part="1"
-AR Path="/60799273/607587D5" Ref="#PWR?"  Part="1"
-AR Path="/607F6DB5/607587D5" Ref="#PWR?"  Part="1"
-AR Path="/6072B375/607587D5" Ref="#PWR0148"  Part="1"
-F 0 "#PWR0148" H 5050 1850 50  0001 C CNN
-F 1 "+3V3" H 4950 2150 50  0000 C CNN
-F 2 "" H 5050 2000 50  0001 C CNN
-F 3 "" H 5050 2000 50  0001 C CNN
-	1    5050 2000
-	1    0    0    -1
-$EndComp
-$Comp
 L power:GND #PWR?
 U 1 1 607587DD
@@
 Wire Wire Line
 	5050 2000 5150 2000
+$Comp
+L power:+3V3_2 #PWR0151
+U 1 1 61235220
+P 3800 1700
+F 0 "#PWR0151" H 3800 1550 50  0001 C CNN
+F 1 "+3V3_2" H 3815 1873 50  0000 C CNN
+F 2 "" H 3800 1700 50  0001 C CNN
+F 3 "" H 3800 1700 50  0001 C CNN
+	1    3800 1700
+	1    0    0    -1
+$EndComp
+Connection ~ 3800 1700
+$Comp
+L power:+3V3_2 #PWR0153
+U 1 1 612355AE
+P 5050 2000
+F 0 "#PWR0153" H 5050 1850 50  0001 C CNN
+F 1 "+3V3_2" H 4900 2150 50  0000 C CNN
+F 2 "" H 5050 2000 50  0001 C CNN
+F 3 "" H 5050 2000 50  0001 C CNN
+	1    5050 2000
+	1    0    0    -1
+$EndComp
 Connection ~ 5050 2000
+$Comp
+L power:+3V3_2 #PWR0161
+U 1 1 61235EDE
+P 5400 1450
+F 0 "#PWR0161" H 5400 1300 50  0001 C CNN
+F 1 "+3V3_2" H 5250 1600 50  0000 C CNN
+F 2 "" H 5400 1450 50  0001 C CNN
+F 3 "" H 5400 1450 50  0001 C CNN
+	1    5400 1450
+	1    0    0    -1
+$EndComp
 $EndSCHEMATC
