File: MCU_3.sch (KiCad schematic (older format))
At the start: 18 parts, among them U9 STM32F051K6Ux

Commit message: Lots of routing done
Connections:
- net labels added: +3V3_1
- net labels removed: +3V3
Changed lines of the file:
@@
 $EndComp
 $Comp
-L power:+3V3 #PWR?
-U 1 1 60308078
-P 3800 1700
-AR Path="/60308078" Ref="#PWR?"  Part="1"
-AR Path="/60302A40/60308078" Ref="#PWR0101"  Part="1"
-AR Path="/605793E5/60308078" Ref="#PWR0149"  Part="1"
-AR Path="/6057AB62/60308078" Ref="#PWR0178"  Part="1"
-AR Path="/60597D10/60308078" Ref="#PWR?"  Part="1"
-AR Path="/60568CD3/60308078" Ref="#PWR0193"  Part="1"
-AR Path="/60595215/60308078" Ref="#PWR0193"  Part="1"
-AR Path="/605CA831/60308078" Ref="#PWR0193"  Part="1"
-AR Path="/605DC779/60308078" Ref="#PWR0222"  Part="1"
-AR Path="/60535FFC/60308078" Ref="#PWR0180"  Part="1"
-AR Path="/6055186B/60308078" Ref="#PWR0207"  Part="1"
-AR Path="/6072B375/60308078" Ref="#PWR0138"  Part="1"
-F 0 "#PWR0180" H 3800 1550 50  0001 C CNN
-F 1 "+3V3" H 3815 1873 50  0000 C CNN
-F 2 "" H 3800 1700 50  0001 C CNN
-F 3 "" H 3800 1700 50  0001 C CNN
-	1    3800 1700
-	1    0    0    -1
-$EndComp
-$Comp
 L power:GND #PWR?
 U 1 1 6030807E
@@
 	1    0    0    -1
 $EndComp
-Connection ~ 3800 1700
 Connection ~ 3800 1900
 Wire Wire Line
@@
 NRST
 $Comp
-L power:+3V3 #PWR0110
-U 1 1 605D8EB0
-P 5400 1450
-AR Path="/60302A40/605D8EB0" Ref="#PWR0110"  Part="1"
-AR Path="/605793E5/605D8EB0" Ref="#PWR0157"  Part="1"
-AR Path="/6057AB62/605D8EB0" Ref="#PWR0186"  Part="1"
-AR Path="/60597D10/605D8EB0" Ref="#PWR?"  Part="1"
-AR Path="/60568CD3/605D8EB0" Ref="#PWR0201"  Part="1"
-AR Path="/60595215/605D8EB0" Ref="#PWR0201"  Part="1"
-AR Path="/605CA831/605D8EB0" Ref="#PWR0201"  Part="1"
-AR Path="/605DC779/605D8EB0" Ref="#PWR0230"  Part="1"
-AR Path="/60535FFC/605D8EB0" Ref="#PWR0188"  Part="1"
-AR Path="/6055186B/605D8EB0" Ref="#PWR0219"  Part="1"
-AR Path="/6072B375/605D8EB0" Ref="#PWR0145"  Part="1"
-F 0 "#PWR0188" H 5400 1300 50  0001 C CNN
-F 1 "+3V3" H 5300 1600 50  0000 C CNN
-F 2 "" H 5400 1450 50  0001 C CNN
-F 3 "" H 5400 1450 50  0001 C CNN
-	1    5400 1450
-	1    0    0    -1
-$EndComp
-$Comp
 L Device:C_Small C?
 U 1 1 605D8EBD
@@
 AR Path="/6072B375/6056C29D" Ref="#PWR0149"  Part="1"
 F 0 "#PWR0162" H 6100 1400 50  0001 C CNN
-F 1 "+3V3A_3" H 6085 1623 50  0000 C CNN
+F 1 "+3V3A_3" H 6250 1600 50  0000 C CNN
 F 2 "" H 6100 1450 50  0001 C CNN
 F 3 "" H 6100 1450 50  0001 C CNN
@@
 $EndComp
 $Comp
-L power:+3V3 #PWR?
-U 1 1 607810C8
-P 5050 2050
-AR Path="/60302A40/607810C8" Ref="#PWR?"  Part="1"
-AR Path="/605793E5/607810C8" Ref="#PWR?"  Part="1"
-AR Path="/6054D32F/607810C8" Ref="#PWR?"  Part="1"
-AR Path="/605CA831/607810C8" Ref="#PWR?"  Part="1"
-AR Path="/6073F35C/607810C8" Ref="#PWR?"  Part="1"
-AR Path="/60799273/607810C8" Ref="#PWR?"  Part="1"
-AR Path="/607F6DB5/607810C8" Ref="#PWR?"  Part="1"
-AR Path="/6072B375/607810C8" Ref="#PWR?"  Part="1"
-AR Path="/60535FFC/607810C8" Ref="#PWR0179"  Part="1"
-F 0 "#PWR0179" H 5050 1900 50  0001 C CNN
-F 1 "+3V3" H 4950 2200 50  0000 C CNN
-F 2 "" H 5050 2050 50  0001 C CNN
-F 3 "" H 5050 2050 50  0001 C CNN
-	1    5050 2050
-	1    0    0    -1
-$EndComp
-$Comp
 L power:+3V3A_3 #PWR0156
 U 1 1 6078E7EF
@@
 Wire Wire Line
 	5050 2050 5150 2050
+$Comp
+L power:+3V3_1 #PWR0205
+U 1 1 61237C9D
+P 3800 1700
+F 0 "#PWR0205" H 3800 1550 50  0001 C CNN
+F 1 "+3V3_1" H 3815 1873 50  0000 C CNN
+F 2 "" H 3800 1700 50  0001 C CNN
+F 3 "" H 3800 1700 50  0001 C CNN
+	1    3800 1700
+	1    0    0    -1
+$EndComp
+Connection ~ 3800 1700
+$Comp
+L power:+3V3_1 #PWR0206
+U 1 1 612382DD
+P 5050 2050
+F 0 "#PWR0206" H 5050 1900 50  0001 C CNN
+F 1 "+3V3_1" H 5065 2223 50  0000 C CNN
+F 2 "" H 5050 2050 50  0001 C CNN
+F 3 "" H 5050 2050 50  0001 C CNN
+	1    5050 2050
+	1    0    0    -1
+$EndComp
 Connection ~ 5050 2050
+$Comp
+L power:+3V3_1 #PWR0213
+U 1 1 612387A6
+P 5400 1450
+F 0 "#PWR0213" H 5400 1300 50  0001 C CNN
+F 1 "+3V3_1" H 5250 1600 50  0000 C CNN
+F 2 "" H 5400 1450 50  0001 C CNN
+F 3 "" H 5400 1450 50  0001 C CNN
+	1    5400 1450
+	1    0    0    -1
+$EndComp
 $EndSCHEMATC
