File: F051-ESC-6L-V1.kicad_pcb (KiCad board)
At the start: 4 copper layers, 46 x 55.8 mm, 222 parts, among them J1 Conn_01x02, J10 Conn_01x03, J11 Conn_01x03, J2 Conn_01x10, J3 Conn_01x04, J4 Conn_01x04, J5 Conn_01x04, J6 Conn_01x03, J7 Conn_01x04, J8 Conn_01x03, J9 Conn_01x10, Q1 TPH1R204PB, Q10 TPH1R204PB, Q11 TPH1R204PB, Q12 TPH1R204PB, Q13 TPH1R204PB, Q14 TPH1R204PB, Q15 TPH1R204PB, Q16 TPH1R204PB, Q17 TPH1R204PB, Q18 TPH1R204PB, Q19 TPH1R204PB, Q2 TPH1R204PB, Q20 TPH1R204PB, Q21 TPH1R204PB, Q22 TPH1R204PB, Q23 TPH1R204PB, Q24 TPH1R204PB, Q3 TPH1R204PB, Q4 TPH1R204PB, Q5 TPH1R204PB, Q6 TPH1R204PB, Q7 TPH1R204PB, Q8 TPH1R204PB, Q9 TPH1R204PB, U1 FD6288Q, U10 FD6288Q, U11 FD6288Q, U12 STM32F051K6Ux, U13 L78L12_SOT89, U14 MP4462, U15 DTOM, U2 STM32F051K6Ux, U3 L78L12_SOT89, U4 LP2985-3.3, U5 INA139, U6 STM32F051K6Ux, U7 OPA340NA, U8 FD6288Q, U9 STM32F051K6Ux

Commit message: Lots of routing done
Parts:
- added C73: 1uF, Capacitor_SMD:C_0402_1005Metric, F.Cu at (144.5, 79.0)
- added C77: 10nF, Capacitor_SMD:C_0402_1005Metric, F.Cu at (145.5, 80.4)
- added C78: 2.2uF, Capacitor_SMD:C_0603_1608Metric, F.Cu at (144.3, 81.0)
- added U16: LP2985-3.3, Package_TO_SOT_SMD:SOT-23-5, F.Cu at (141.8, 80.4)
- moved C22 8.55 mm to (135.5, 79.0), turned to 180 degrees
- moved C24 8.31 mm to (135.7, 81.0)
- moved R52 7.91 mm to (129.5, 96.4)
- moved C23 4.66 mm to (134.5, 80.4)
- moved R60 4.21 mm to (130.1, 86.3), turned to 270 degrees
- moved R12 3.89 mm to (149.9, 90.7), turned to 90 degrees
- moved U4 3.32 mm to (138.2, 80.4)
- moved R11 1.97 mm to (149.9, 88.8)
- moved R59 1.91 mm to (130.1, 88.1)
- moved C69 1.89 mm to (134.9, 97.4), turned to 180 degrees
- moved C4 1.64 mm to (140.9, 97.9)
- moved R10 1.10 mm to (149.9, 94.0)
- moved U15 1.10 mm to (140.1, 89.8)
- moved R51 1.03 mm to (129.9, 97.8)
- moved J10 1.00 mm to (119.0, 81.5)
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Connections:
- C13 pad 1: +3V3 -> +3V3_2
- C14 pad 1: +3V3 -> +3V3_2
- C23 pad 1: +3V3 -> +3V3_1
- C24 pad 1: +3V3 -> +3V3_1
- C25 pad 1: +3V3 -> +3V3_2
- C26 pad 1: +3V3 -> +3V3_2
- C34 pad 1: +3V3 -> +3V3_1
- C35 pad 1: +3V3 -> +3V3_1
- C47 pad 1: +3V3 -> +3V3_1
- C48 pad 1: +3V3 -> +3V3_1
- FB1 pad 2: +3V3 -> +3V3_2
- FB2 pad 2: +3V3 -> +3V3_2
- FB3 pad 2: +3V3 -> +3V3_1
- FB4 pad 2: +3V3 -> +3V3_1
- U12 pad 1: +3V3 -> +3V3_1
- U12 pad 17: +3V3 -> +3V3_1
- U2 pad 1: +3V3 -> +3V3_2
- U2 pad 17: +3V3 -> +3V3_2
- U4 pad 4: +3V3 -> +3V3_1
- U4 pad 5: +3V3 -> +3V3_1
- U6 pad 1: +3V3 -> +3V3_2
- U6 pad 17: +3V3 -> +3V3_2
- U7 pad 5: +3V3 -> +3V3_2
- U9 pad 1: +3V3 -> +3V3_1
- U9 pad 17: +3V3 -> +3V3_1
Routing:
- net +3V3: track 99.8 -> 0.00 mm, vias 14 -> 0
- net /Curent Sense/CURR: track 46.6 -> 6.35 mm, vias 3 -> 1
- net /PWM_1: track 43.3 -> 6.51 mm, vias 3 -> 1
- net +12V_2: track 35.7 -> 4.91 mm, vias 8 -> 2
- net /PWM_2: track 30.8 -> 6.68 mm, vias 3 -> 1
- net /PWM_3: track 30.0 -> 6.85 mm, vias 3 -> 1
- net VCC_Shunt: track 16.2 -> 2.69 mm, vias 124 -> 79
- net +3V3_1: track 0.00 -> 11.9 mm, vias 0 -> 7
- net /MCU_4/PhaseB: track 27.5 -> 18.8 mm, vias 17 -> 16
- net /MOSFET Driver 3/LO2: track 1.34 -> 10.0 mm, vias 0 -> 2
- net /MCU_1/USART1_RX: track 18.5 -> 10.2 mm
- net /MCU 3/PhaseA: track 30.8 -> 23.6 mm, vias 16 -> 17
- net /MCU_2/SWDIO: track 15.2 -> 8.74 mm
- net /MCU_2/PhaseC: track 24.7 -> 18.5 mm
- net /MOSFET_Driver_4/LO3: track 1.81 -> 7.71 mm, vias 0 -> 2
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- added copper zone on F.Cu, net +12V_1
- added copper zone on In4.Cu, net +12V_1
- added copper zone on In4.Cu, net +12V_2
- added copper zone on F.Cu, net +3V3_1
- added copper zone on In4.Cu, net +3V3_1
- added copper zone on F.Cu, net +3V3_2
- added copper zone on In2.Cu, net GND
- added copper zone on In3.Cu, net GND
- added copper zone on F.Cu, net Net-(C75-Pad1)
- added copper zone on F.Cu, net Net-(R73-Pad2)
- added copper zone on In4.Cu, net VCC_Shunt
- removed copper zone on In2.Cu, net +12V_1
- removed copper zone on In2.Cu, net +12V_2
- removed copper zone on F.Cu, net +3V3
- removed copper zone on In2.Cu, net /PWM_2
- removed copper zone on In2.Cu, net VCC_Shunt
Other:
- copper layers 4 -> 6
- net class Default: clearance 0.1 -> 0.127; trace_width 0.1 -> 0.127; via_dia 0.45 -> 0.4572; via_drill 0.2 -> 0.254
- net class Min removed
- net class OshPark added: clearance 0.127, trace_width 0.127, via_dia 0.4572, via_drill 0.254
- rule trace_clearance: 0.1 -> 0.127
- rule trace_min: 0.1 -> 0.127
- rule via_min_drill: 0.2 -> 0.254
- rule via_min_size: 0.45 -> 0.4572

Commit message: More routing done
Parts:
- moved J11 1.00 mm to (119.0, 95.5)
- moved J6 1.00 mm to (161.0, 95.5)
- moved J8 1.00 mm to (161.0, 81.5)
Routing:
- net /Curent Sense/CURR: track 6.35 -> 45.9 mm, vias 1 -> 2
- net /PWM_1: track 6.51 -> 44.6 mm, vias 1 -> 2
- net +12V_2: track 4.91 -> 32.9 mm, vias 2 -> 9
- net /PWM_3: track 6.85 -> 29.6 mm, vias 1 -> 2
- net /PWM_2: track 6.68 -> 29.2 mm, vias 1 -> 2
- net +3V3_2: track 5.20 -> 18.5 mm, vias 0 -> 9
- net /MCU_4/PhaseB: track 18.8 -> 27.3 mm, vias 16 -> 17
- net VCC_Shunt: track 2.69 -> 8.79 mm, vias 79 -> 81
- net /MCU 3/PhaseC: track 21.6 -> 18.0 mm
- net +12V_1: track 32.6 -> 35.7 mm
- net /MOSFET_Driver_1/LO3: track 7.25 -> 5.97 mm
- net /MOSFET_Driver_2/VB1: track 11.0 -> 12.2 mm
- net /MCU_1/PhaseA: track 27.2 -> 28.2 mm
- net /MCU_4/USART1_TX: track 10.6 -> 11.4 mm
- net /MCU_1/SWDIO: track 12.7 -> 13.4 mm
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- added copper zone on In4.Cu, net +3V3_2
- removed copper zone on F.Cu, net +12V_1

Commit message: Finished routing
Parts:
- moved R52 0.64 mm to (129.0, 96.8), turned to 90 degrees
Routing:
- net VCC_Shunt: track 8.79 -> 17.2 mm, vias 81 -> 89
- net +3V3_1: track 11.9 -> 15.7 mm
- net /MCU_4/PhaseA: track 25.3 -> 23.1 mm, vias 16 -> 23
- net /MOSFET Driver 3/LO2: track 10.0 -> 11.2 mm
- net Net-(Q16-Pad4): track 4.38 -> 3.38 mm
- net +12V_1: track 35.7 -> 36.4 mm
- net Net-(Q15-Pad4): track 12.0 -> 11.5 mm
- net /MCU_2/USART1_RX: track 10.1 -> 10.6 mm
- net /MOSFET_Driver_2/VB1: track 12.2 -> 12.5 mm, vias 2 -> 3
- net /MCU_1/PhaseA: track 28.2 -> 27.9 mm, vias 16 -> 23
- net /MCU 3/PhaseC: vias 15 -> 22
- net GND: vias 72 -> 138
- net /MCU_2/PhaseC: vias 15 -> 22
- added copper zone on Power, net +12V_1
- added copper zone on Power, net +12V_2
- added copper zone on Power, net +3V3_1
- added copper zone on Power, net +3V3_2
- added copper zone on Signal_2, net /MCU 3/PhaseC
- added copper zone on Signal_3, net /MCU 3/PhaseC
- added copper zone on Signal_2, net /MCU_1/PhaseA
- added copper zone on Signal_3, net /MCU_1/PhaseA
- added copper zone on Signal_2, net /MCU_2/PhaseC
- added copper zone on Signal_3, net /MCU_2/PhaseC
- added copper zone on Signal_2, net /MCU_4/PhaseA
- added copper zone on Signal_3, net /MCU_4/PhaseA
- added copper zone on GND, net GND
- added copper zone on Signal_2, net GND
- added copper zone on Signal_3, net GND
- added copper zone on B.Cu, net VCC_Shunt
- added copper zone on Power, net VCC_Shunt
- removed copper zone on In4.Cu, net +12V_1
- removed copper zone on In4.Cu, net +12V_2
- removed copper zone on In4.Cu, net +3V3_1
- removed copper zone on In4.Cu, net +3V3_2
- removed copper zone on In1.Cu, net GND
- removed copper zone on In2.Cu, net GND
- removed copper zone on In3.Cu, net GND
- removed copper zone on In4.Cu, net VCC_Shunt

Commit message: Added PNGs and PDFs
Parts:
- moved R71 0.20 mm to (130.6, 75.0)
Routing:
- net /MCU 3/PhaseC: track 18.0 -> 21.8 mm, vias 22 -> 19
- net /MCU_2/PhaseC: track 18.6 -> 22.3 mm, vias 22 -> 19
- net /MCU_4/USART1_TX: track 11.4 -> 13.6 mm
- net /MCU 3/PhaseA: track 23.6 -> 25.3 mm, vias 17 -> 21
- net /MCU_4/PhaseA: track 23.1 -> 21.7 mm, vias 23 -> 19
- net VCC_Shunt: track 17.2 -> 15.8 mm, vias 89 -> 93
- net +12V_1: track 36.4 -> 37.7 mm
- net +12V_2: track 32.9 -> 34.1 mm
- net /MOSFET Driver 3/VB1: track 10.7 -> 9.52 mm
- net /MCU_4/USART1_RX: track 10.5 -> 11.6 mm
- net Net-(Q20-Pad4): track 10.1 -> 11.0 mm
- net /MOSFET_Driver_2/VB1: track 12.5 -> 13.2 mm
- net /MOSFET_Driver_1/VB1: track 11.1 -> 10.5 mm
- net /MCU_4/PhaseC: track 25.1 -> 24.5 mm, vias 15 -> 19
- net Net-(Q2-Pad4): track 10.7 -> 11.2 mm
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- added copper zone on Signal_2, net /MCU 3/PhaseA
- added copper zone on Signal_3, net /MCU 3/PhaseA
- added copper zone on Signal_2, net /MCU 3/PhaseB
- added copper zone on Signal_3, net /MCU 3/PhaseB
- added copper zone on Signal_2, net /MCU_1/PhaseB
- added copper zone on Signal_3, net /MCU_1/PhaseB
- added copper zone on Signal_2, net /MCU_1/PhaseC
- added copper zone on Signal_3, net /MCU_1/PhaseC
- added copper zone on Signal_2, net /MCU_2/PhaseA
- added copper zone on Signal_3, net /MCU_2/PhaseA
- added copper zone on Signal_2, net /MCU_2/PhaseB
- added copper zone on Signal_3, net /MCU_2/PhaseB
- added copper zone on Signal_2, net /MCU_4/PhaseB
- added copper zone on Signal_3, net /MCU_4/PhaseB
- added copper zone on Signal_2, net /MCU_4/PhaseC
- added copper zone on Signal_3, net /MCU_4/PhaseC
Other:
- board text added: "JEREMY WOLFE"
- board text removed: "MIDN WOLFE"
