File: F051-ESC-6L-V1.sch (KiCad schematic (older format))
At the start: 40 parts, among them J1 Conn_01x02, J10 Conn_01x03, J11 Conn_01x03, J2 Conn_01x10, J3 Conn_01x04, J4 Conn_01x04, J5 Conn_01x04, J6 Conn_01x03, J7 Conn_01x04, J8 Conn_01x03, J9 Conn_01x10, U15 DTOM

Commit message: Added PNGs and PDFs
Other:
- note added: "Main Sheet"
- moved on the sheet: C16, C17, C18, C19, C20, C21, C50, C51, C52, C53, C54, C55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
